File: 2634482 - Denardi Zoe - Microduino/2634482 - Denardi Zoe - Microduino.kicad_pcb (KiCad board)
At the start: 2 copper layers, 33.5 x 30.5 mm, 14 parts, among them J1 USB_A_UCC, J2 Conn_01x10_Socket, U1 ATtiny85-20S

Commit message: Entrega final
Parts:
- moved J1 10.5 mm to (132.0, 45.5)
Routing:
- net GND: track 88.5 -> 99.5 mm
- net Net-(D5-K): track 21.4 -> 31.0 mm
- net Net-(D1-A): track 16.2 -> 6.91 mm
- net Net-(D2-K): track 20.5 -> 18.9 mm
- net Net-(J2-Pin_8): track 30.8 -> 30.0 mm
- net Net-(J2-Pin_7): track 24.0 -> 24.6 mm
Other:
- outline, holes or cut-outs redrawn
